File: Hardware/MaD_Board/KICAD/MAD_Board.sch (KiCad schematic (older format))
At the start: 73 parts, among them J1 Conn_02x05_Odd_Even, J10 Conn_01x05, J2 Conn_02x05_Odd_Even, J3 Conn_02x05_Odd_Even, J4 Conn_02x05_Odd_Even, J5 Conn_02x03_Odd_Even, J7 Power, J8 USB_B_Micro, J9 Micro_SD_Card, P10 CONN_01X01, P11 CONN_01X01, P12 CONN_01X01, P13 CONN_01X01, P2 Power, P3 Analog, P4 Analog, P5 PWM, P6 PWM, P7 Communication, P8 CONN_01X01, P9 CONN_01X01, Q1 MMBT3904, SW1 SW_Push, U1 P8X32A-Q44, U2 SPX2920T-5.0_TO263, U3 AT24C512, U4 FT232RL, U5 AMS1117-3.3, U6 LMV321, U7 APM4953

Commit message: groundwork for p2
Parts:
- removed C12, C7: 4.7uF, Capacitor_SMD:C_0603_1608Metric, symbol Device:C_Small
- removed C13, C8: 1uF, Capacitor_SMD:C_0603_1608Metric, symbol Device:C_Small
- removed C5, C6: 10uF, Capacitor_SMD:C_0805_2012Metric, symbol Device:C_Small
- removed U2: SPX2920T-5.0_TO263, Package_TO_SOT_SMD:TO-263-3_TabPin2, symbol Regulator_Linear:SPX2920T-5.0_TO263
- removed U5: AMS1117-3.3, Package_TO_SOT_SMD:SOT-223-3_TabPin2, symbol Regulator_Linear:AMS1117-3.3
- added C? (x2): 1uF, Capacitor_SMD:C_0603_1608Metric, symbol Device:C_Small
- added C? (x2): 4.7uF, Capacitor_SMD:C_0603_1608Metric, symbol Device:C_Small
- added C? (x2): 10uF, Capacitor_SMD:C_0805_2012Metric, symbol Device:C_Small
- added U?: AMS1117-3.3, Package_TO_SOT_SMD:SOT-223-3_TabPin2, symbol Regulator_Linear:AMS1117-3.3
- added U?: SPX2920T-5.0_TO263, Package_TO_SOT_SMD:TO-263-3_TabPin2, symbol Regulator_Linear:SPX2920T-5.0_TO263
Connections:
- net +3V3: now also C?.1, C?.1, U?.2 (VO)
- net +5V: now also C?.1, C?.1, C?.2, U?.3 (VI), U?.3 (VO)
- net GND: now also C?.1, C?.1, C?.2, C?.2, C?.2, C?.2, U?.1 (GND), U?.2 (GND)
- net VIN: now also C?.2, U?.1 (VI)
