File: Hardware/MAD_P2/MAD_P2.sch (KiCad schematic (older format))
At the start: 52 parts

Commit message: Created power system for the MAD_P2 board, using evaluation board as reference
Parts:
- removed C? (x8): 470uF, symbol Device:C_Small
- removed C? (x4): 180uF, symbol Device:C_Small
- removed C? (x4): 330uF, symbol Device:C_Small
- removed D? (x8): SS36, symbol Device:D_Schottky_Small
- removed J? (x3): Conn_01x02, symbol Connector_Generic:Conn_01x02
- removed JP?: Jumper_1_3.3V, symbol Jumper:Jumper_2_Open
- removed JP?: Jumper_1_5V, symbol Jumper:Jumper_2_Open
- removed JP?: Jumper_1_VIN, symbol Jumper:Jumper_2_Open
- removed JP?: Jumper_2_3.3V, symbol Jumper:Jumper_2_Open
- removed JP?: Jumper_2_5V, symbol Jumper:Jumper_2_Open
- removed JP?: Jumper_2_VIN, symbol Jumper:Jumper_2_Open
- removed JP?: Jumper_3_3.3V, symbol Jumper:Jumper_2_Open
- removed JP?: Jumper_3_5V, symbol Jumper:Jumper_2_Open
- removed JP?: Jumper_3_VIN, symbol Jumper:Jumper_2_Open
- removed L? (x4): 68uH/3A, symbol Device:L_Small
- removed L? (x4): 47uH/3A, symbol Device:L_Small
- removed U? (x4): XL1509-5.0, symbol MAD_Board:XL1509
- removed U? (x4): XL1509-3.3, symbol MAD_Board:XL1509
- added C1, C11, C12, C13, C15, C17, C18, C19, C21, C23, C24, C25, C27, C29, C3, C30, C31, C33, C35, C36, C37, C39, C41, C42, C43, C45, C47, C48, C5, C6, C7, C9: 4.7uF, symbol Device:C_Small
- added C10, C14, C16, C2, C20, C22, C26, C28, C32, C34, C38, C4, C40, C44, C46, C8: 1uF, symbol Device:C_Small
- added U1: P2X8C4M64P-REF, symbol P2X8C4M64P:P2X8C4M64P-REF
- added Y1: 20MHz, symbol Device:Crystal_GND24_Small
Connections:
- net labels added: +1V8, P0, P1, P10, P11, P12, P13, P14, P15, P16, P17, P18, P19, P2, P20, P21, P22, P23, P24, P25, P26, P27, P28, P29, P3, P30, P31, P32, P33, P34, P35, P36, P37, P38, P39, P4, P40, P41, P42, P43, P44, P45, P46, P47, P48, P49, P5, P50, P51, P52, P53, P54, P55, P56, P57, P58, P59, P6, P60, P61, P62, P63, P7, P8, P9, V_0_3, V_12_15, V_16_19, V_20_23, V_24_27, V_28_31, V_32_35, V_36_39, V_40_43, V_44_47, V_48_51, V_4_7, V_52_55, V_56_59, V_60_63, V_8_11
- net labels removed: +3.3V, +3.3V_1, +3.3V_2, +3.3V_3, +5V, +5V_1, +5V_2, +5V_3, VIN
- wire segments 135 -> 70
Other:
- note added: "Core Supply Capacitors"
- note added: "IO Supply Capacitors"
- note removed: "Line Out #1"
- note removed: "Line Out #2"
- note removed: "Line Out #3"
- note removed: "Main Board Power"

Commit message: Added memory and usb to schematic
Parts:
- added R?: 10K, symbol Device:R_Small
Connections:
- net labels added: RESET
- wire segments 70 -> 73
Changed lines of the file:
@@
 $Descr A4 11693 8268
 encoding utf-8
-Sheet 1 3
+Sheet 1 5
 Title "MaD_P2"
 Date "2021-05-06"
@@
 	4500 1900 4600 1900
 $Sheet
-S -2100 3150 1950 1150
+S -2150 1150 1950 1150
 U 60E5FA00
 F0 "Power" 50
@@
 $EndSheet
 $Sheet
-S -2100 4650 1950 1000
+S -2150 2650 1950 1000
 U 60F79100
 F0 "IO Power" 50
@@
 Wire Wire Line
 	9500 3150 9900 3150
+$Sheet
+S -2150 4050 1950 900
+U 60B0DD34
+F0 "Memory" 50
+F1 "Memory.sch" 50
+$EndSheet
+$Comp
+L Device:R_Small R?
+U 1 1 60B1E34F
+P 2650 5850
+F 0 "R?" V 2846 5850 50  0000 C CNN
+F 1 "10K" V 2755 5850 50  0000 C CNN
+F 2 "" H 2650 5850 50  0001 C CNN
+F 3 "~" H 2650 5850 50  0001 C CNN
+	1    2650 5850
+	0    -1   -1   0
+$EndComp
+Wire Wire Line
+	2850 5300 2850 5850
+Wire Wire Line
+	2850 5850 2750 5850
+Text Label 2350 5850 2    50   ~ 0
+V_56_59
+Wire Wire Line
+	2550 5850 2350 5850
+$Sheet
+S -2150 5300 1950 850
+U 60B76FA1
+F0 "USB" 50
+F1 "USB.sch" 50
+$EndSheet
+Text Label 2850 5350 3    50   ~ 0
+RESET
 $EndSCHEMATC

Commit message: Added wifi to board
Other:
- moved on the sheet: R?, Y1

Commit message: added adc
Parts:
- U1: symbol P2X8C4M64P:P2X8C4M64P-REF -> MAD_P2-rescue:P2X8C4M64P-REF-P2X8C4M64P
Other:
- note added: "Propeller 2"
- moved on the sheet: C1, C10, C13, C14, C15, C16, C19, C2, C20, C21, C22, C25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

Commit message: finished adc, added dac
Connections:
- wire segments 73 -> 74
Changed lines of the file:
@@
 $Descr A4 11693 8268
 encoding utf-8
-Sheet 1 6
+Sheet 1 7
 Title "MaD_P2"
 Date "2021-05-06"
@@
 Text Notes 2950 2050 0    129  ~ 0
 Propeller 2
+$Sheet
+S -2150 7500 1950 900
+U 60C11A52
+F0 "PeripheralsCont" 50
+F1 "PeripheralsCont.sch" 50
+$EndSheet
+Wire Wire Line
+	-1050 7800 -1050 7750
 $EndSCHEMATC

Commit message: began pcb layout
Parts:
- C1, C10, C11, C12, C13, C14, C15, C16, C17, C18, C19, C2, C20, C21, C22, C23, C24, C25, C26, C27, C28, C29, C3, C30, C31, C32, C33, C34, C35, C36, C37, C38, C39, C4, C40, C41, C42, C43, C44, C45, C46, C47, C48, C5, C6, C7, C8, C9: footprint (none) -> Capacitor_SMD:C_0603_1608Metric
- R2: renamed from R?; footprint (none) -> Resistor_SMD:R_0603_1608Metric
- U1: footprint (none) -> Package_QFP:TQFP-100-1EP_14x14mm_P0.5mm_EP5x5mm_ThermalVias
- Y1: footprint (none) -> Crystal:Crystal_SMD_3225-4Pin_3.2x2.5mm
Connections:
- wire segments 74 -> 73

Commit message: added lcsc part numbers to bom
Parts:
- C1, C11, C12, C13, C15, C17, C18, C19, C21, C23, C24, C25, C27, C29, C3, C30, C31, C33, C35, C36, C37, C39, C41, C42, C43, C45, C47, C48, C5, C6, C7, C9: LCSC (none) -> C19666; TYPE (none) -> BASIC
- C10, C14, C16, C2, C20, C22, C26, C28, C32, C34, C38, C4, C40, C44, C46, C8: LCSC (none) -> C15849; TYPE (none) -> BASIC
- R2: LCSC (none) -> C25804; TYPE (none) -> BASIC
- U1: TYPE (none) -> NA
- Y1: LCSC (none) -> C172730; TYPE (none) -> EXT
