File: Hardware/MAD_P2/Peripherals.sch (KiCad schematic (older format))
At the start: 84 parts, among them J12 Micro_SD_Card, U28 DS3231M, U29 ESP-12F, U30 ADS131E08-REF

Commit message: added lcsc part numbers to bom
Parts:
- BT1: LCSC (none) -> C70377; TYPE (none) -> EXT
- C108, C110, C112, C113, C116: LCSC (none) -> C15849; TYPE (none) -> BASIC
- C109, C111, C114, C117: LCSC (none) -> C14663; TYPE (none) -> BASIC
- C115: LCSC (none) -> C59461; TYPE (none) -> BASIC
- C118: footprint Capacitor_SMD:C_0603_1608Metric -> Capacitor_SMD:C_0805_2012Metric; LCSC (none) -> C15850; TYPE (none) -> EXT
- C119, C120, C121, C122, C123, C124, C125, C126, C127, C128, C129, C130, C131, C132, C133, C134: LCSC (none) -> C1620; TYPE (none) -> BASIC
- J12: LCSC (none) -> C397369; TYPE (none) -> CHK
- JP18, JP19, JP20, JP21, R30, TP1, TP10, TP11, TP12, TP13, TP14, TP15, TP16, TP2, TP3, TP4, TP5, TP6, TP7, TP8, TP9, U30: TYPE (none) -> NA
- R23, R24, R26, R27, R29, R31, R32, R33, R34, R35, R36, R37, R38, R39, R40, R41, R42, R43, R44, R45, R46, R47, R48, R49, R50, R51, R52, R53, R54: LCSC (none) -> C25804; TYPE (none) -> BASIC
- R25: LCSC (none) -> C23350; TYPE (none) -> BASIC
- R28: LCSC (none) -> C23179; TYPE (none) -> BASIC
- U28: LCSC (none) -> C9866; TYPE (none) -> EXT
- U29: LCSC (none) -> C82891; TYPE (none) -> EXT
