File: Hardware/MAD_P2/PeripheralsCont.sch (KiCad schematic (older format))
At the start: 6 parts

Commit message: began pcb layout
Parts:
- C135, C136, C137, C138, C139: renamed from C?; footprint (none) -> Capacitor_SMD:C_0603_1608Metric
- U31: renamed from U?; footprint (none) -> Package_SO:TSSOP-16_4.4x5mm_P0.65mm
Changed lines of the file:
@@
 $EndDescr
 $Comp
-L MAD_P2-rescue:MAX5134-7 U?
+L MAD_P2-rescue:MAX5134-7 U31
 U 1 1 60C13D6D
 P 1900 1900
-F 0 "U?" H 1900 2350 50  0000 C CNN
+F 0 "U31" H 1900 2350 50  0000 C CNN
 F 1 "MAX5134-7" H 1850 1450 50  0000 C CNN
-F 2 "" H 1950 1900 50  0001 C CNN
+F 2 "Package_SO:TSSOP-16_4.4x5mm_P0.65mm" H 1950 1900 50  0001 C CNN
 F 3 "" H 1950 1900 50  0001 C CNN
 	1    1900 1900
@@
 	2250 1350 2250 1550
 $Comp
-L Device:C_Small C?
+L Device:C_Small C135
 U 1 1 60C1568C
 P 1900 1250
-F 0 "C?" H 1992 1296 50  0000 L CNN
+F 0 "C135" H 1992 1296 50  0000 L CNN
 F 1 "47pF" H 1992 1205 50  0000 L CNN
-F 2 "" H 1900 1250 50  0001 C CNN
+F 2 "Capacitor_SMD:C_0603_1608Metric" H 1900 1250 50  0001 C CNN
 F 3 "~" H 1900 1250 50  0001 C CNN
 	1    1900 1250
@@
 	1900 1350 2250 1350
 $Comp
-L power:GND #PWR?
+L power:GND #PWR0211
 U 1 1 60C16203
 P 1900 1150
-F 0 "#PWR?" H 1900 900 50  0001 C CNN
+F 0 "#PWR0211" H 1900 900 50  0001 C CNN
 F 1 "GND" H 1905 977 50  0000 C CNN
 F 2 "" H 1900 1150 50  0001 C CNN
@@
 P 1200 2250
 AR Path="/609BFBB9/60C3F571" Ref="#PWR?"  Part="1"
-AR Path="/60C11A52/60C3F571" Ref="#PWR?"  Part="1"
-F 0 "#PWR?" H 1200 2000 50  0001 C CNN
+AR Path="/60C11A52/60C3F571" Ref="#PWR0212"  Part="1"
+F 0 "#PWR0212" H 1200 2000 50  0001 C CNN
 F 1 "GND" H 1205 2077 50  0000 C CNN
 F 2 "" H 1200 2250 50  0001 C CNN
@@
 P 2400 1650
 AR Path="/609BFBB9/60C4089F" Ref="#PWR?"  Part="1"
-AR Path="/60C11A52/60C4089F" Ref="#PWR?"  Part="1"
-F 0 "#PWR?" H 2400 1400 50  0001 C CNN
+AR Path="/60C11A52/60C4089F" Ref="#PWR0213"  Part="1"
+F 0 "#PWR0213" H 2400 1400 50  0001 C CNN
 F 1 "GND" V 2405 1522 50  0000 R CNN
 F 2 "" H 2400 1650 50  0001 C CNN
@@
 P 2400 1850
 AR Path="/609BFBB9/60C47B17" Ref="#PWR?"  Part="1"
-AR Path="/60C11A52/60C47B17" Ref="#PWR?"  Part="1"
-F 0 "#PWR?" H 2400 1600 50  0001 C CNN
+AR Path="/60C11A52/60C47B17" Ref="#PWR0214"  Part="1"
+F 0 "#PWR0214" H 2400 1600 50  0001 C CNN
 F 1 "GND" V 2405 1722 50  0000 R CNN
 F 2 "" H 2400 1850 50  0001 C CNN
@@
 3.3V_ADC
 $Comp
-L Device:C_Small C?
+L Device:C_Small C136
 U 1 1 60C48DE5
 P 2450 1250
-F 0 "C?" H 2542 1296 50  0000 L CNN
+F 0 "C136" H 2542 1296 50  0000 L CNN
 F 1 "0.1uF" H 2542 1205 50  0000 L CNN
-F 2 "" H 2450 1250 50  0001 C CNN
+F 2 "Capacitor_SMD:C_0603_1608Metric" H 2450 1250 50  0001 C CNN
 F 3 "~" H 2450 1250 50  0001 C CNN
 	1    2450 1250
@@
 $EndComp
 $Comp
-L Device:C_Small C?
+L Device:C_Small C137
 U 1 1 60C497BA
 P 2900 1250
-F 0 "C?" H 2992 1296 50  0000 L CNN
+F 0 "C137" H 2992 1296 50  0000 L CNN
 F 1 "4.7uF" H 2992 1205 50  0000 L CNN
-F 2 "" H 2900 1250 50  0001 C CNN
+F 2 "Capacitor_SMD:C_0603_1608Metric" H 2900 1250 50  0001 C CNN
 F 3 "~" H 2900 1250 50  0001 C CNN
 	1    2900 1250
@@
 P 2700 1400
 AR Path="/609BFBB9/60C4A300" Ref="#PWR?"  Part="1"
-AR Path="/60C11A52/60C4A300" Ref="#PWR?"  Part="1"
-F 0 "#PWR?" H 2700 1150 50  0001 C CNN
+AR Path="/60C11A52/60C4A300" Ref="#PWR0215"  Part="1"
+F 0 "#PWR0215" H 2700 1150 50  0001 C CNN
 F 1 "GND" H 2705 1227 50  0000 C CNN
 F 2 "" H 2700 1400 50  0001 C CNN
@@
 3.3V_ADC
 $Comp
-L Device:C_Small C?
+L Device:C_Small C138
 U 1 1 60C4E119
 P 3300 1250
-F 0 "C?" H 3392 1296 50  0000 L CNN
+F 0 "C138" H 3392 1296 50  0000 L CNN
 F 1 "0.1uF" H 3392 1205 50  0000 L CNN
-F 2 "" H 3300 1250 50  0001 C CNN
+F 2 "Capacitor_SMD:C_0603_1608Metric" H 3300 1250 50  0001 C CNN
 F 3 "~" H 3300 1250 50  0001 C CNN
 	1    3300 1250
@@
 $EndComp
 $Comp
-L Device:C_Small C?
+L Device:C_Small C139
 U 1 1 60C4E11F
 P 3750 1250
-F 0 "C?" H 3842 1296 50  0000 L CNN
+F 0 "C139" H 3842 1296 50  0000 L CNN
 F 1 "4.7uF" H 3842 1205 50  0000 L CNN
-F 2 "" H 3750 1250 50  0001 C CNN
+F 2 "Capacitor_SMD:C_0603_1608Metric" H 3750 1250 50  0001 C CNN
 F 3 "~" H 3750 1250 50  0001 C CNN
 	1    3750 1250
@@
 P 3550 1400
 AR Path="/609BFBB9/60C4E128" Ref="#PWR?"  Part="1"
-AR Path="/60C11A52/60C4E128" Ref="#PWR?"  Part="1"
-F 0 "#PWR?" H 3550 1150 50  0001 C CNN
+AR Path="/60C11A52/60C4E128" Ref="#PWR0216"  Part="1"
+F 0 "#PWR0216" H 3550 1150 50  0001 C CNN
 F 1 "GND" H 3555 1227 50  0000 C CNN
 F 2 "" H 3550 1400 50  0001 C CNN

Commit message: added lcsc part numbers to bom
Parts:
- C135: LCSC (none) -> C1671; TYPE (none) -> BASIC
- C136, C138: LCSC (none) -> C14663; TYPE (none) -> BASIC
- C137, C139: LCSC (none) -> C19666; TYPE (none) -> BASIC
- U31: LCSC (none) -> C143511; TYPE (none) -> EXT
Changed lines of the file:
@@
 F 2 "Package_SO:TSSOP-16_4.4x5mm_P0.65mm" H 1950 1900 50  0001 C CNN
 F 3 "" H 1950 1900 50  0001 C CNN
+F 4 "C143511" H 1900 1900 50  0001 C CNN "LCSC"
+F 5 "EXT" H 1900 1900 50  0001 C CNN "TYPE"
 	1    1900 1900
 	1    0    0    -1
@@
 F 2 "Capacitor_SMD:C_0603_1608Metric" H 1900 1250 50  0001 C CNN
 F 3 "~" H 1900 1250 50  0001 C CNN
+F 4 "C1671" H 1900 1250 50  0001 C CNN "LCSC"
+F 5 "BASIC" H 1900 1250 50  0001 C CNN "TYPE"
 	1    1900 1250
 	1    0    0    -1
@@
 F 2 "Capacitor_SMD:C_0603_1608Metric" H 2450 1250 50  0001 C CNN
 F 3 "~" H 2450 1250 50  0001 C CNN
+F 4 "C14663" H 2450 1250 50  0001 C CNN "LCSC"
+F 5 "BASIC" H 2450 1250 50  0001 C CNN "TYPE"
 	1    2450 1250
 	1    0    0    -1
@@
 F 2 "Capacitor_SMD:C_0603_1608Metric" H 2900 1250 50  0001 C CNN
 F 3 "~" H 2900 1250 50  0001 C CNN
+F 4 "C19666" H 2900 1250 50  0001 C CNN "LCSC"
+F 5 "BASIC" H 2900 1250 50  0001 C CNN "TYPE"
 	1    2900 1250
 	1    0    0    -1
@@
 F 2 "Capacitor_SMD:C_0603_1608Metric" H 3300 1250 50  0001 C CNN
 F 3 "~" H 3300 1250 50  0001 C CNN
+F 4 "C14663" H 3300 1250 50  0001 C CNN "LCSC"
+F 5 "BASIC" H 3300 1250 50  0001 C CNN "TYPE"
 	1    3300 1250
 	1    0    0    -1
@@
 F 2 "Capacitor_SMD:C_0603_1608Metric" H 3750 1250 50  0001 C CNN
 F 3 "~" H 3750 1250 50  0001 C CNN
+F 4 "C19666" H 3750 1250 50  0001 C CNN "LCSC"
+F 5 "BASIC" H 3750 1250 50  0001 C CNN "TYPE"
 	1    3750 1250
 	1    0    0    -1
