File: Hardware/MAD_P2/PeripheralsCont.sch (KiCad schematic (older format))
At the start: 6 parts, among them U31 MAX5134-7

Commit message: replaced ads131E with ads131A
Parts:
- removed C135: 47pF, Capacitor_SMD:C_0603_1608Metric, symbol Device:C_Small
- removed C136, C138: 0.1uF, Capacitor_SMD:C_0603_1608Metric, symbol Device:C_Small
- removed C137, C139: 4.7uF, Capacitor_SMD:C_0603_1608Metric, symbol Device:C_Small
- removed U31: MAX5134-7, Package_SO:TSSOP-16_4.4x5mm_P0.65mm, symbol MAD_P2-rescue:MAX5134-7
Connections:
- no-connect marks 1 -> 0
Other:
- note removed: "16 Bit DAC"
Changed lines of the file:
@@
 Comment4 ""
 $EndDescr
-$Comp
-L MAD_P2-rescue:MAX5134-7 U31
-U 1 1 60C13D6D
-P 1900 1900
-F 0 "U31" H 1900 2350 50  0000 C CNN
-F 1 "MAX5134-7" H 1850 1450 50  0000 C CNN
-F 2 "Package_SO:TSSOP-16_4.4x5mm_P0.65mm" H 1950 1900 50  0001 C CNN
-F 3 "" H 1950 1900 50  0001 C CNN
-	1    1900 1900
-	1    0    0    -1
-$EndComp
-Wire Wire Line
-	1500 1550 1500 1350
-Wire Wire Line
-	1500 1350 1900 1350
-Wire Wire Line
-	2250 1350 2250 1550
-$Comp
-L Device:C_Small C135
-U 1 1 60C1568C
-P 1900 1250
-F 0 "C135" H 1992 1296 50  0000 L CNN
-F 1 "47pF" H 1992 1205 50  0000 L CNN
-F 2 "Capacitor_SMD:C_0603_1608Metric" H 1900 1250 50  0001 C CNN
-F 3 "~" H 1900 1250 50  0001 C CNN
-	1    1900 1250
-	1    0    0    -1
-$EndComp
-Connection ~ 1900 1350
-Wire Wire Line
-	1900 1350 2250 1350
-$Comp
-L power:GND #PWR0211
-U 1 1 60C16203
-P 1900 1150
-F 0 "#PWR0211" H 1900 900 50  0001 C CNN
-F 1 "GND" H 1905 977 50  0000 C CNN
-F 2 "" H 1900 1150 50  0001 C CNN
-F 3 "" H 1900 1150 50  0001 C CNN
-	1    1900 1150
-	-1   0    0    1
-$EndComp
-Text Label 2250 2250 0    50   ~ 0
-P48
-Text Label 2250 2150 0    50   ~ 0
-P49
-Text Label 1500 2250 2    50   ~ 0
-P50
-$Comp
-L power:GND #PWR?
-U 1 1 60C3F571
-P 1200 2250
-AR Path="/609BFBB9/60C3F571" Ref="#PWR?"  Part="1"
-AR Path="/60C11A52/60C3F571" Ref="#PWR0212"  Part="1"
-F 0 "#PWR0212" H 1200 2000 50  0001 C CNN
-F 1 "GND" H 1205 2077 50  0000 C CNN
-F 2 "" H 1200 2250 50  0001 C CNN
-F 3 "" H 1200 2250 50  0001 C CNN
-	1    1200 2250
-	1    0    0    -1
-$EndComp
-Wire Wire Line
-	1200 2250 1200 2150
-Wire Wire Line
-	1200 2150 1500 2150
-NoConn ~ 1500 1950
-$Comp
-L power:GND #PWR?
-U 1 1 60C4089F
-P 2400 1650
-AR Path="/609BFBB9/60C4089F" Ref="#PWR?"  Part="1"
-AR Path="/60C11A52/60C4089F" Ref="#PWR0213"  Part="1"
-F 0 "#PWR0213" H 2400 1400 50  0001 C CNN
-F 1 "GND" V 2405 1522 50  0000 R CNN
-F 2 "" H 2400 1650 50  0001 C CNN
-F 3 "" H 2400 1650 50  0001 C CNN
-	1    2400 1650
-	0    -1   -1   0
-$EndComp
-Text GLabel 1500 1850 0    50   Input ~ 0
-3.3V_ADC
-Text GLabel 1500 1650 0    50   Input ~ 0
-3.3V_ADC
-Text Label 1500 2050 2    50   ~ 0
-A03
-Text Label 2250 2050 0    50   ~ 0
-A02
-Text Label 2250 1750 0    50   ~ 0
-A01
-$Comp
-L power:GND #PWR?
-U 1 1 60C47B17
-P 2400 1850
-AR Path="/609BFBB9/60C47B17" Ref="#PWR?"  Part="1"
-AR Path="/60C11A52/60C47B17" Ref="#PWR0214"  Part="1"
-F 0 "#PWR0214" H 2400 1600 50  0001 C CNN
-F 1 "GND" V 2405 1722 50  0000 R CNN
-F 2 "" H 2400 1850 50  0001 C CNN
-F 3 "" H 2400 1850 50  0001 C CNN
-	1    2400 1850
-	0    -1   -1   0
-$EndComp
-Wire Wire Line
-	2250 1650 2400 1650
-Wire Wire Line
-	2250 1850 2400 1850
-Text GLabel 2700 1050 1    50   Input ~ 0
-3.3V_ADC
-$Comp
-L Device:C_Small C136
-U 1 1 60C48DE5
-P 2450 1250
-F 0 "C136" H 2542 1296 50  0000 L CNN
-F 1 "0.1uF" H 2542 1205 50  0000 L CNN
-F 2 "Capacitor_SMD:C_0603_1608Metric" H 2450 1250 50  0001 C CNN
-F 3 "~" H 2450 1250 50  0001 C CNN
-	1    2450 1250
-	1    0    0    -1
-$EndComp
-$Comp
-L Device:C_Small C137
-U 1 1 60C497BA
-P 2900 1250
-F 0 "C137" H 2992 1296 50  0000 L CNN
-F 1 "4.7uF" H 2992 1205 50  0000 L CNN
-F 2 "Capacitor_SMD:C_0603_1608Metric" H 2900 1250 50  0001 C CNN
-F 3 "~" H 2900 1250 50  0001 C CNN
-	1    2900 1250
-	1    0    0    -1
-$EndComp
-Wire Wire Line
-	2450 1050 2450 1150
-Wire Wire Line
-	2900 1050 2900 1150
-Wire Wire Line
-	2450 1050 2900 1050
-$Comp
-L power:GND #PWR?
-U 1 1 60C4A300
-P 2700 1400
-AR Path="/609BFBB9/60C4A300" Ref="#PWR?"  Part="1"
-AR Path="/60C11A52/60C4A300" Ref="#PWR0215"  Part="1"
-F 0 "#PWR0215" H 2700 1150 50  0001 C CNN
-F 1 "GND" H 2705 1227 50  0000 C CNN
-F 2 "" H 2700 1400 50  0001 C CNN
-F 3 "" H 2700 1400 50  0001 C CNN
-	1    2700 1400
-	1    0    0    -1
-$EndComp
-Wire Wire Line
-	2450 1350 2450 1400
-Wire Wire Line
-	2450 1400 2700 1400
-Wire Wire Line
-	2900 1350 2900 1400
-Wire Wire Line
-	2900 1400 2700 1400
-Connection ~ 2700 1400
-Text GLabel 3550 1050 1    50   Input ~ 0
-3.3V_ADC
-$Comp
-L Device:C_Small C138
-U 1 1 60C4E119
-P 3300 1250
-F 0 "C138" H 3392 1296 50  0000 L CNN
-F 1 "0.1uF" H 3392 1205 50  0000 L CNN
-F 2 "Capacitor_SMD:C_0603_1608Metric" H 3300 1250 50  0001 C CNN
-F 3 "~" H 3300 1250 50  0001 C CNN
-	1    3300 1250
-	1    0    0    -1
-$EndComp
-$Comp
-L Device:C_Small C139
-U 1 1 60C4E11F
-P 3750 1250
-F 0 "C139" H 3842 1296 50  0000 L CNN
-F 1 "4.7uF" H 3842 1205 50  0000 L CNN
-F 2 "Capacitor_SMD:C_0603_1608Metric" H 3750 1250 50  0001 C CNN
-F 3 "~" H 3750 1250 50  0001 C CNN
-	1    3750 1250
-	1    0    0    -1
-$EndComp
-Wire Wire Line
-	3300 1050 3300 1150
-Wire Wire Line
-	3750 1050 3750 1150
-Wire Wire Line
-	3300 1050 3750 1050
-$Comp
-L power:GND #PWR?
-U 1 1 60C4E128
-P 3550 1400
-AR Path="/609BFBB9/60C4E128" Ref="#PWR?"  Part="1"
-AR Path="/60C11A52/60C4E128" Ref="#PWR0216"  Part="1"
-F 0 "#PWR0216" H 3550 1150 50  0001 C CNN
-F 1 "GND" H 3555 1227 50  0000 C CNN
-F 2 "" H 3550 1400 50  0001 C CNN
-F 3 "" H 3550 1400 50  0001 C CNN
-	1    3550 1400
-	1    0    0    -1
-$EndComp
-Wire Wire Line
-	3300 1350 3300 1400
-Wire Wire Line
-	3300 1400 3550 1400
-Wire Wire Line
-	3750 1350 3750 1400
-Wire Wire Line
-	3750 1400 3550 1400
-Connection ~ 3550 1400
-Text Notes 1650 750  2    129  ~ 0
-16 Bit DAC
-Text GLabel 2450 1950 2    50   Input ~ 0
-3.3V_ADC
-Wire Wire Line
-	2450 1950 2250 1950
 $EndSCHEMATC
