File: Hardware/MAD_P2/Connections.sch (KiCad schematic (older format))
At the start: 49 parts, among them J10 Conn_02x05_Odd_Even, J11 Conn_02x05_Odd_Even, J13 Conn_02x05_Odd_Even, J14 Conn_02x05_Odd_Even, J15 Conn_ADC1, J16 Conn_DAC, J18 P3, J19 P4, J20 P2, J21 Conn_02x05_Odd_Even, J22 Conn_02x05_Odd_Even, J23 Conn_02x03_Odd_Even, J24 P5, J25 P6, J26 P7, J31 Micro_SD_Card_Connector, J32 Micro_SD_Card_Socket, J34 FTDI 1x6, J6 Edge_Conn, J7 Conn_02x05_Odd_Even, J8 USB_C_Receptacle_USB2.0, J9 Conn_02x05_Odd_Even, Q1 MMBT3904, U27 FT232RL

Commit message: updated bom with lcsc part #
Parts:
- J10, J11, J13, J14, J21, J22, J7, J9: LCSC (none) -> C5665; TYPE NA -> EXT
- J15, J16: LCSC (none) -> C5665; TYPE DIGIKEY -> EXT
- J18, J19, J20, J25, J26: LCSC (none) -> C27438; TYPE AMAZON -> EXT
- J23: LCSC (none) -> C92272; TYPE AMAZON -> EXT
- J24: LCSC (none) -> C35445; TYPE AMAZON -> EXT
- J31: LCSC (none) -> C293349; TYPE DIGIKEY -> EXT
- J32: LCSC (none) -> C719027; TYPE DIGIKEY -> EXT
- J34: TYPE (none) -> NA
- J8: LCSC C165948 -> C393939
Changed lines of the file:
@@
 F 2 "Connector_USB:USB_C_Receptacle_Palconn_UTC16-G" H 3100 2500 50  0001 C CNN
 F 3 "https://www.usb.org/sites/default/files/documents/usb_type-c.zip" H 3100 2500 50  0001 C CNN
-F 4 "C165948" H 2950 2500 50  0001 C CNN "LCSC"
+F 4 "C393939" H 2950 2500 50  0001 C CNN "LCSC"
 F 5 "EXT" H 2950 2500 50  0001 C CNN "TYPE"
 	1    2950 2500
@@
 F 2 "Connector_IDC:IDC-Header_2x05_P2.54mm_Vertical" H 4800 7250 50  0001 C CNN
 F 3 "~" H 4800 7250 50  0001 C CNN
-F 4 "NA" H 4800 7250 50  0001 C CNN "TYPE"
+F 4 "EXT" H 4800 7250 50  0001 C CNN "TYPE"
+F 5 "C5665" H 4800 7250 50  0001 C CNN "LCSC"
 	1    4800 7250
 	0    -1   -1   0
@@
 F 2 "Connector_IDC:IDC-Header_2x05_P2.54mm_Vertical" H 4050 7250 50  0001 C CNN
 F 3 "~" H 4050 7250 50  0001 C CNN
-F 4 "NA" H 4050 7250 50  0001 C CNN "TYPE"
+F 4 "EXT" H 4050 7250 50  0001 C CNN "TYPE"
+F 5 "C5665" H 4050 7250 50  0001 C CNN "LCSC"
 	1    4050 7250
 	0    -1   -1   0
@@
 F 2 "Connector_IDC:IDC-Header_2x05_P2.54mm_Vertical" H 3250 7250 50  0001 C CNN
 F 3 "~" H 3250 7250 50  0001 C CNN
-F 4 "NA" H 3250 7250 50  0001 C CNN "TYPE"
+F 4 "EXT" H 3250 7250 50  0001 C CNN "TYPE"
+F 5 "C5665" H 3250 7250 50  0001 C CNN "LCSC"
 	1    3250 7250
 	0    -1   -1   0
@@
 F 2 "Connector_IDC:IDC-Header_2x05_P2.54mm_Vertical" H 2450 7250 50  0001 C CNN
 F 3 "~" H 2450 7250 50  0001 C CNN
-F 4 "NA" H 2450 7250 50  0001 C CNN "TYPE"
+F 4 "EXT" H 2450 7250 50  0001 C CNN "TYPE"
+F 5 "C5665" H 2450 7250 50  0001 C CNN "LCSC"
 	1    2450 7250
 	0    -1   -1   0
@@
 F 2 "Connector_IDC:IDC-Header_2x05_P2.54mm_Vertical" H 4900 5550 50  0001 C CNN
 F 3 "~" H 4900 5550 50  0001 C CNN
-F 4 "NA" H 4900 5550 50  0001 C CNN "TYPE"
+F 4 "EXT" H 4900 5550 50  0001 C CNN "TYPE"
+F 5 "C5665" H 4900 5550 50  0001 C CNN "LCSC"
 	1    4900 5550
 	0    -1   -1   0
@@
 F 2 "Connector_IDC:IDC-Header_2x05_P2.54mm_Vertical" H 4050 5400 50  0001 C CNN
 F 3 "~" H 4050 5400 50  0001 C CNN
-F 4 "NA" H 4050 5400 50  0001 C CNN "TYPE"
+F 4 "EXT" H 4050 5400 50  0001 C CNN "TYPE"
+F 5 "C5665" H 4050 5400 50  0001 C CNN "LCSC"
 	1    4050 5400
 	0    -1   -1   0
@@
 F 2 "Connector_IDC:IDC-Header_2x05_P2.54mm_Vertical" H 3400 5400 50  0001 C CNN
 F 3 "~" H 3400 5400 50  0001 C CNN
-F 4 "NA" H 3400 5400 50  0001 C CNN "TYPE"
+F 4 "EXT" H 3400 5400 50  0001 C CNN "TYPE"
+F 5 "C5665" H 3400 5400 50  0001 C CNN "LCSC"
 	1    3400 5400
 	0    -1   -1   0
@@
 F 2 "Connector_IDC:IDC-Header_2x05_P2.54mm_Vertical" H 2750 5400 50  0001 C CNN
 F 3 "~" H 2750 5400 50  0001 C CNN
-F 4 "NA" H 2750 5400 50  0001 C CNN "TYPE"
+F 4 "EXT" H 2750 5400 50  0001 C CNN "TYPE"
+F 5 "C5665" H 2750 5400 50  0001 C CNN "LCSC"
 	1    2750 5400
 	0    -1   -1   0
@@
 F 3 "~" H 9800 1450 50  0001 C CNN
 F 4 "S9169-ND" H 9800 1450 50  0001 C CNN "DIGIKEY"
-F 5 "DIGIKEY" H 9800 1450 50  0001 C CNN "TYPE"
+F 5 "EXT" H 9800 1450 50  0001 C CNN "TYPE"
+F 6 "C5665" H 9800 1450 50  0001 C CNN "LCSC"
 	1    9800 1450
 	0    -1   -1   0
@@
 F 3 "~" H 9950 3100 50  0001 C CNN
 F 4 "S9169-ND" H 9950 3100 50  0001 C CNN "DIGIKEY"
-F 5 "DIGIKEY" H 9950 3100 50  0001 C CNN "TYPE"
+F 5 "EXT" H 9950 3100 50  0001 C CNN "TYPE"
+F 6 "C5665" H 9950 3100 50  0001 C CNN "LCSC"
 	1    9950 3100
 	0    -1   -1   0
@@
 F 2 "Connector_PinSocket_2.54mm:PinSocket_1x08_P2.54mm_Vertical" H 9450 4200 50  0001 C CNN
 F 3 "~" H 9450 4200 50  0001 C CNN
-F 4 "AMAZON" H 9450 4200 50  0001 C CNN "TYPE"
+F 4 "EXT" H 9450 4200 50  0001 C CNN "TYPE"
+F 5 "C27438" H 9450 4200 50  0001 C CNN "LCSC"
 	1    9450 4200
 	1    0    0    -1
@@
 F 2 "Connector_PinSocket_2.54mm:PinSocket_1x08_P2.54mm_Vertical" H 9100 5100 50  0001 C CNN
 F 3 "~" H 9100 5100 50  0001 C CNN
-F 4 "AMAZON" H 9100 5100 50  0001 C CNN "TYPE"
+F 4 "EXT" H 9100 5100 50  0001 C CNN "TYPE"
+F 5 "C27438" H 9100 5100 50  0001 C CNN "LCSC"
 	1    9100 5100
 	1    0    0    -1
@@
 F 2 "Connector_PinSocket_2.54mm:PinSocket_1x08_P2.54mm_Vertical" H 9100 6000 50  0001 C CNN
 F 3 "~" H 9100 6000 50  0001 C CNN
-F 4 "AMAZON" H 9100 6000 50  0001 C CNN "TYPE"
+F 4 "EXT" H 9100 6000 50  0001 C CNN "TYPE"
+F 5 "C27438" H 9100 6000 50  0001 C CNN "LCSC"
 	1    9100 6000
 	1    0    0    -1
@@
 F 2 "Connector_PinSocket_2.54mm:PinSocket_1x08_P2.54mm_Vertical" H 10400 6050 50  0001 C CNN
 F 3 "~" H 10400 6050 50  0001 C CNN
-F 4 "AMAZON" H 10400 6050 50  0001 C CNN "TYPE"
+F 4 "EXT" H 10400 6050 50  0001 C CNN "TYPE"
+F 5 "C27438" H 10400 6050 50  0001 C CNN "LCSC"
 	1    10400 6050
 	-1   0    0    -1
@@
 F 2 "Connector_PinSocket_2.54mm:PinSocket_1x10_P2.54mm_Vertical" H 10400 4250 50  0001 C CNN
 F 3 "~" H 10400 4250 50  0001 C CNN
-F 4 "AMAZON" H 10400 4250 50  0001 C CNN "TYPE"
+F 4 "EXT" H 10400 4250 50  0001 C CNN "TYPE"
+F 5 "C35445" H 10400 4250 50  0001 C CNN "LCSC"
 	1    10400 4250
 	-1   0    0    -1
@@
 F 2 "Connector_PinSocket_2.54mm:PinSocket_2x03_P2.54mm_Vertical" H 9700 5800 50  0001 C CNN
 F 3 "~" H 9700 5800 50  0001 C CNN
-F 4 "AMAZON" H 9700 5800 50  0001 C CNN "TYPE"
+F 4 "EXT" H 9700 5800 50  0001 C CNN "TYPE"
+F 5 "C92272" H 9700 5800 50  0001 C CNN "LCSC"
 	1    9700 5800
 	-1   0    0    -1
@@
 F 2 "Connector_PinSocket_2.54mm:PinSocket_1x08_P2.54mm_Vertical" H 10400 5200 50  0001 C CNN
 F 3 "~" H 10400 5200 50  0001 C CNN
-F 4 "AMAZON" H 10400 5200 50  0001 C CNN "TYPE"
+F 4 "EXT" H 10400 5200 50  0001 C CNN "TYPE"
+F 5 "C27438" H 10400 5200 50  0001 C CNN "LCSC"
 	1    10400 5200
 	-1   0    0    -1
@@
 F 3 "http://katalog.we-online.de/em/datasheet/693072010801.pdf" H 7800 4550 50  0001 C CNN
 F 4 "WM26501" H 7800 4550 50  0001 C CNN "DIGIKEY"
-F 5 "DIGIKEY" H 7800 4550 50  0001 C CNN "TYPE"
+F 5 "EXT" H 7800 4550 50  0001 C CNN "TYPE"
+F 6 "C293349" H 7800 4550 50  0001 C CNN "LCSC"
 	1    7800 4550
 	1    0    0    -1
@@
 F 3 "http://katalog.we-online.de/em/datasheet/693072010801.pdf" H 7800 5800 50  0001 C CNN
 F 4 "732-3820-2-ND" H 7800 5800 50  0001 C CNN "DIGIKEY"
-F 5 "DIGIKEY" H 7800 5800 50  0001 C CNN "TYPE"
+F 5 "EXT" H 7800 5800 50  0001 C CNN "TYPE"
+F 6 "C719027" H 7800 5800 50  0001 C CNN "LCSC"
 	1    7800 5800
 	1    0    0    -1
@@
 F 2 "Connector_PinHeader_2.54mm:PinHeader_1x06_P2.54mm_Vertical" H 4600 3050 50  0001 C CNN
 F 3 "~" H 4600 3050 50  0001 C CNN
+F 4 "NA" H 4600 3050 50  0001 C CNN "TYPE"
 	1    4600 3050
 	1    0    0    -1

Commit message: added more functionality to JSON for motion quartet, motion set, motion profiles, machine profile, and more
Parts:
- C103, C104, C105, C106, C107, D12, D9, J8, Q1, R1, R14, R15, R16, R17, R18, R19, R20, R21, R22, R35, R36: ASSEMBLED (none) -> YES
- F4, J10, J11, J13, J14, J15, J16, J18, J19, J20, J21, J22, J23, J24, J25, J26, J31, J32, J7, J9, U27: ASSEMBLED (none) -> NO
Changed lines of the file:
@@
 F 4 "C15850" H 7050 1200 50  0001 C CNN "LCSC"
 F 5 "BASIC" H 7050 1200 50  0001 C CNN "TYPE"
+F 6 "YES" H 7050 1200 50  0001 C CNN "ASSEMBLED"
 	1    7050 1200
 	1    0    0    -1
@@
 F 4 "C14663" H 6550 1200 50  0001 C CNN "LCSC"
 F 5 "BASIC" H 6550 1200 50  0001 C CNN "TYPE"
+F 6 "YES" H 6550 1200 50  0001 C CNN "ASSEMBLED"
 	1    6550 1200
 	1    0    0    -1
@@
 F 4 "C25190" H 3700 2650 50  0001 C CNN "LCSC"
 F 5 "BASIC" H 3700 2650 50  0001 C CNN "TYPE"
+F 6 "YES" H 3700 2650 50  0001 C CNN "ASSEMBLED"
 	1    3700 2650
 	0    -1   -1   0
@@
 F 4 "C25190" H 3700 2450 50  0001 C CNN "LCSC"
 F 5 "BASIC" H 3700 2450 50  0001 C CNN "TYPE"
+F 6 "YES" H 3700 2450 50  0001 C CNN "ASSEMBLED"
 	1    3700 2450
 	0    1    1    0
@@
 F 4 "C20526" H 8050 2200 50  0001 C CNN "LCSC"
 F 5 "BASIC" H 8050 2200 50  0001 C CNN "TYPE"
+F 6 "YES" H 8050 2200 50  0001 C CNN "ASSEMBLED"
 	1    8050 2200
 	1    0    0    -1
@@
 F 4 "C25804" H 7700 2300 50  0001 C CNN "LCSC"
 F 5 "BASIC" H 7700 2300 50  0001 C CNN "TYPE"
+F 6 "YES" H 7700 2300 50  0001 C CNN "ASSEMBLED"
 	1    7700 2300
 	-1   0    0    1
@@
 F 4 "C57112" H 7450 2200 50  0001 C CNN "LCSC"
 F 5 "BASIC" H 7450 2200 50  0001 C CNN "TYPE"
+F 6 "YES" H 7450 2200 50  0001 C CNN "ASSEMBLED"
 	1    7450 2200
 	0    1    1    0
@@
 F 4 "C23350" H 7150 1900 50  0001 C CNN "LCSC"
 F 5 "BASIC" H 7150 1900 50  0001 C CNN "TYPE"
+F 6 "YES" H 7150 1900 50  0001 C CNN "ASSEMBLED"
 	1    7150 1900
 	0    1    -1   0
@@
 F 4 "C23350" H 7150 1800 50  0001 C CNN "LCSC"
 F 5 "BASIC" H 7150 1800 50  0001 C CNN "TYPE"
+F 6 "YES" H 7150 1800 50  0001 C CNN "ASSEMBLED"
 	1    7150 1800
 	0    -1   1    0
@@
 F 4 "C21190" H 7750 2900 50  0001 C CNN "LCSC"
 F 5 "BASIC" H 7750 2900 50  0001 C CNN "TYPE"
+F 6 "YES" H 7750 2900 50  0001 C CNN "ASSEMBLED"
 	1    7750 2900
 	0    1    -1   0
@@
 F 4 "C21190" H 7750 2800 50  0001 C CNN "LCSC"
 F 5 "BASIC" H 7750 2800 50  0001 C CNN "TYPE"
+F 6 "YES" H 7750 2800 50  0001 C CNN "ASSEMBLED"
 	1    7750 2800
 	0    1    1    0
@@
 F 4 "C72043" H 7450 2900 50  0001 C CNN "LCSC"
 F 5 "BASIC" H 7450 2900 50  0001 C CNN "TYPE"
+F 6 "YES" H 7450 2900 50  0001 C CNN "ASSEMBLED"
 	1    7450 2900
 	1    0    0    -1
@@
 F 4 "C72041" H 7250 2800 50  0001 C CNN "LCSC"
 F 5 "BASIC" H 7250 2800 50  0001 C CNN "TYPE"
+F 6 "YES" H 7250 2800 50  0001 C CNN "ASSEMBLED"
 	1    7250 2800
 	1    0    0    -1
@@
 F 4 "C57112" H 4650 1550 50  0001 C CNN "LCSC"
 F 5 "BASIC" H 4650 1550 50  0001 C CNN "TYPE"
+F 6 "YES" H 4650 1550 50  0001 C CNN "ASSEMBLED"
 	1    4650 1550
 	1    0    0    -1
@@
 F 4 "C14663" H 5050 1900 50  0001 C CNN "LCSC"
 F 5 "BASIC" H 5050 1900 50  0001 C CNN "TYPE"
+F 6 "YES" H 5050 1900 50  0001 C CNN "ASSEMBLED"
 	1    5050 1900
 	1    0    0    -1
@@
 F 4 "C8690" H 6150 2500 50  0001 C CNN "LCSC"
 F 5 "BASIC" H 6150 2500 50  0001 C CNN "TYPE"
+F 6 "NO" H 6150 2500 50  0001 C CNN "ASSEMBLED"
 	1    6150 2500
 	1    0    0    -1
@@
 F 4 "C23186" H 4400 2200 50  0001 C CNN "LCSC"
 F 5 "BASIC" H 4400 2200 50  0001 C CNN "TYPE"
+F 6 "YES" H 4400 2200 50  0001 C CNN "ASSEMBLED"
 	1    4400 2200
 	0    1    1    0
@@
 F 4 "C23186" H 4100 2100 50  0001 C CNN "LCSC"
 F 5 "BASIC" H 4100 2100 50  0001 C CNN "TYPE"
+F 6 "YES" H 4100 2100 50  0001 C CNN "ASSEMBLED"
 	1    4100 2100
 	0    1    1    0
@@
 F 4 "C261937" H 3800 1650 50  0001 C CNN "LCSC"
 F 5 "EXT" H 3800 1650 50  0001 C CNN "TYPE"
+F 6 "NO" H 3800 1650 50  0001 C CNN "ASSEMBLED"
 	1    3800 1650
 	1    0    0    -1
@@
 F 4 "C393939" H 2950 2500 50  0001 C CNN "LCSC"
 F 5 "EXT" H 2950 2500 50  0001 C CNN "TYPE"
+F 6 "YES" H 2950 2500 50  0001 C CNN "ASSEMBLED"
 	1    2950 2500
 	1    0    0    -1
@@
 F 4 "EXT" H 4800 7250 50  0001 C CNN "TYPE"
 F 5 "C5665" H 4800 7250 50  0001 C CNN "LCSC"
+F 6 "NO" H 4800 7250 50  0001 C CNN "ASSEMBLED"
 	1    4800 7250
 	0    -1   -1   0
@@
 F 4 "EXT" H 4050 7250 50  0001 C CNN "TYPE"
 F 5 "C5665" H 4050 7250 50  0001 C CNN "LCSC"
+F 6 "NO" H 4050 7250 50  0001 C CNN "ASSEMBLED"
 	1    4050 7250
 	0    -1   -1   0
@@
 F 4 "EXT" H 3250 7250 50  0001 C CNN "TYPE"
 F 5 "C5665" H 3250 7250 50  0001 C CNN "LCSC"
+F 6 "NO" H 3250 7250 50  0001 C CNN "ASSEMBLED"
 	1    3250 7250
 	0    -1   -1   0
@@
 F 4 "EXT" H 2450 7250 50  0001 C CNN "TYPE"
 F 5 "C5665" H 2450 7250 50  0001 C CNN "LCSC"
+F 6 "NO" H 2450 7250 50  0001 C CNN "ASSEMBLED"
 	1    2450 7250
 	0    -1   -1   0
@@
 F 4 "EXT" H 4900 5550 50  0001 C CNN "TYPE"
 F 5 "C5665" H 4900 5550 50  0001 C CNN "LCSC"
+F 6 "NO" H 4900 5550 50  0001 C CNN "ASSEMBLED"
 	1    4900 5550
 	0    -1   -1   0
@@
 F 4 "EXT" H 4050 5400 50  0001 C CNN "TYPE"
 F 5 "C5665" H 4050 5400 50  0001 C CNN "LCSC"
+F 6 "NO" H 4050 5400 50  0001 C CNN "ASSEMBLED"
 	1    4050 5400
 	0    -1   -1   0
@@
 F 4 "EXT" H 3400 5400 50  0001 C CNN "TYPE"
 F 5 "C5665" H 3400 5400 50  0001 C CNN "LCSC"
+F 6 "NO" H 3400 5400 50  0001 C CNN "ASSEMBLED"
 	1    3400 5400
 	0    -1   -1   0
@@
 F 4 "EXT" H 2750 5400 50  0001 C CNN "TYPE"
 F 5 "C5665" H 2750 5400 50  0001 C CNN "LCSC"
+F 6 "NO" H 2750 5400 50  0001 C CNN "ASSEMBLED"
 	1    2750 5400
 	0    -1   -1   0
@@
 F 5 "EXT" H 9800 1450 50  0001 C CNN "TYPE"
 F 6 "C5665" H 9800 1450 50  0001 C CNN "LCSC"
+F 7 "NO" H 9800 1450 50  0001 C CNN "ASSEMBLED"
 	1    9800 1450
 	0    -1   -1   0
@@
 F 5 "EXT" H 9950 3100 50  0001 C CNN "TYPE"
 F 6 "C5665" H 9950 3100 50  0001 C CNN "LCSC"
+F 7 "NO" H 9950 3100 50  0001 C CNN "ASSEMBLED"
 	1    9950 3100
 	0    -1   -1   0
@@
 F 4 "EXT" H 9450 4200 50  0001 C CNN "TYPE"
 F 5 "C27438" H 9450 4200 50  0001 C CNN "LCSC"
+F 6 "NO" H 9450 4200 50  0001 C CNN "ASSEMBLED"
 	1    9450 4200
 	1    0    0    -1
@@
 F 4 "EXT" H 9100 5100 50  0001 C CNN "TYPE"
 F 5 "C27438" H 9100 5100 50  0001 C CNN "LCSC"
+F 6 "NO" H 9100 5100 50  0001 C CNN "ASSEMBLED"
 	1    9100 5100
 	1    0    0    -1
@@
 F 4 "EXT" H 9100 6000 50  0001 C CNN "TYPE"
 F 5 "C27438" H 9100 6000 50  0001 C CNN "LCSC"
+F 6 "NO" H 9100 6000 50  0001 C CNN "ASSEMBLED"
 	1    9100 6000
 	1    0    0    -1
@@
 F 4 "EXT" H 10400 6050 50  0001 C CNN "TYPE"
 F 5 "C27438" H 10400 6050 50  0001 C CNN "LCSC"
+F 6 "NO" H 10400 6050 50  0001 C CNN "ASSEMBLED"
 	1    10400 6050
 	-1   0    0    -1
@@
 F 4 "EXT" H 10400 4250 50  0001 C CNN "TYPE"
 F 5 "C35445" H 10400 4250 50  0001 C CNN "LCSC"
+F 6 "NO" H 10400 4250 50  0001 C CNN "ASSEMBLED"
 	1    10400 4250
 	-1   0    0    -1
@@
 F 4 "EXT" H 9700 5800 50  0001 C CNN "TYPE"
 F 5 "C92272" H 9700 5800 50  0001 C CNN "LCSC"
+F 6 "NO" H 9700 5800 50  0001 C CNN "ASSEMBLED"
 	1    9700 5800
 	-1   0    0    -1
@@
 F 4 "C25804" H 10900 4750 50  0001 C CNN "LCSC"
 F 5 "BASIC" H 10900 4750 50  0001 C CNN "TYPE"
+F 6 "YES" H 10900 4750 50  0001 C CNN "ASSEMBLED"
 	1    10900 4750
 	0    1    -1   0
@@
 F 4 "EXT" H 10400 5200 50  0001 C CNN "TYPE"
 F 5 "C27438" H 10400 5200 50  0001 C CNN "LCSC"
+F 6 "NO" H 10400 5200 50  0001 C CNN "ASSEMBLED"
 	1    10400 5200
 	-1   0    0    -1
@@
 F 5 "EXT" H 7800 4550 50  0001 C CNN "TYPE"
 F 6 "C293349" H 7800 4550 50  0001 C CNN "LCSC"
+F 7 "NO" H 7800 4550 50  0001 C CNN "ASSEMBLED"
 	1    7800 4550
 	1    0    0    -1
@@
 F 4 "C23350" H 6400 4850 50  0001 C CNN "LCSC"
 F 5 "BASIC" H 6400 4850 50  0001 C CNN "TYPE"
+F 6 "YES" H 6400 4850 50  0001 C CNN "ASSEMBLED"
 	1    6400 4850
 	0    -1   -1   0
@@
 F 5 "EXT" H 7800 5800 50  0001 C CNN "TYPE"
 F 6 "C719027" H 7800 5800 50  0001 C CNN "LCSC"
+F 7 "NO" H 7800 5800 50  0001 C CNN "ASSEMBLED"
 	1    7800 5800
 	1    0    0    -1
@@
 F 4 "C23350" H 6400 6100 50  0001 C CNN "LCSC"
 F 5 "BASIC" H 6400 6100 50  0001 C CNN "TYPE"
+F 6 "YES" H 6400 6100 50  0001 C CNN "ASSEMBLED"
 	1    6400 6100
 	0    -1   -1   0
