File: Hardware/MAD_P2/Power.sch (KiCad schematic (older format))
At the start: 63 parts, among them J4 Power_In, U10 AMS1117-3.3, U11 APM4953, U12 APM4953, U19 AMS1117-1.8, U2 XL1509-5.0, U20 LM321, U21 APM4953, U3 XL1509-5.0, U4 XL1509-5.0, U5 XL1509-5.0, U6 AMS1117-3.3, U7 AMS1117-3.3, U8 AMS1117-3.3, U9 AMS1117-3.3

Commit message: revising pcb layout
Parts:
- F1, F2, F3, F5: renamed from F?; footprint (none) -> Fuse:Fuse_1206_3216Metric
- J4: footprint Connector_AMASS:AMASS_XT30PW-M_1x02_P2.50mm_Horizontal -> MAD_P2:0705530001
Changed lines of the file:
@@
 F 0 "J4" H 9780 1042 50  0000 L CNN
 F 1 "Power_In" H 9780 951 50  0000 L CNN
-F 2 "Connector_AMASS:AMASS_XT30PW-M_1x02_P2.50mm_Horizontal" H 9700 1050 50  0001 C CNN
+F 2 "MAD_P2:0705530001" H 9700 1050 50  0001 C CNN
 F 3 "~" H 9700 1050 50  0001 C CNN
 	1    9700 1050
@@
 Connection ~ 4800 6900
 $Comp
-L Device:Polyfuse_Small F?
+L Device:Polyfuse_Small F1
 U 1 1 60B225D6
 P 8850 2750
-F 0 "F?" V 8645 2750 50  0000 C CNN
+F 0 "F1" V 8645 2750 50  0000 C CNN
 F 1 "5A" V 8736 2750 50  0000 C CNN
-F 2 "" H 8900 2550 50  0001 L CNN
+F 2 "Fuse:Fuse_1206_3216Metric" H 8900 2550 50  0001 L CNN
 F 3 "~" H 8850 2750 50  0001 C CNN
 	1    8850 2750
@@
 $EndComp
 $Comp
-L Device:Polyfuse_Small F?
+L Device:Polyfuse_Small F2
 U 1 1 60B239BA
 P 8900 3850
-F 0 "F?" V 8695 3850 50  0000 C CNN
+F 0 "F2" V 8695 3850 50  0000 C CNN
 F 1 "5A" V 8786 3850 50  0000 C CNN
-F 2 "" H 8950 3650 50  0001 L CNN
+F 2 "Fuse:Fuse_1206_3216Metric" H 8950 3650 50  0001 L CNN
 F 3 "~" H 8900 3850 50  0001 C CNN
 	1    8900 3850
@@
 $EndComp
 $Comp
-L Device:Polyfuse_Small F?
+L Device:Polyfuse_Small F5
 U 1 1 60B24B24
 P 10750 3850
-F 0 "F?" V 10545 3850 50  0000 C CNN
+F 0 "F5" V 10545 3850 50  0000 C CNN
 F 1 "5A" V 10636 3850 50  0000 C CNN
-F 2 "" H 10800 3650 50  0001 L CNN
+F 2 "Fuse:Fuse_1206_3216Metric" H 10800 3650 50  0001 L CNN
 F 3 "~" H 10750 3850 50  0001 C CNN
 	1    10750 3850
@@
 $EndComp
 $Comp
-L Device:Polyfuse_Small F?
+L Device:Polyfuse_Small F3
 U 1 1 60B25972
 P 10750 2800
-F 0 "F?" V 10545 2800 50  0000 C CNN
+F 0 "F3" V 10545 2800 50  0000 C CNN
 F 1 "5A" V 10636 2800 50  0000 C CNN
-F 2 "" H 10800 2600 50  0001 L CNN
+F 2 "Fuse:Fuse_1206_3216Metric" H 10800 2600 50  0001 L CNN
 F 3 "~" H 10750 2800 50  0001 C CNN
 	1    10750 2800

Commit message: completed BOM with digikey and LSCS parts
Parts:
- C140, C141, C142, C57, C58, C59, C60, C62, C71, C88: LCSC (none) -> C19666; TYPE (none) -> BASIC
- C49, C50, C51, C52: DIGIKEY (none) -> 399-18277-1-ND; LCSC (none) -> C3350; TYPE (none) -> EXT
- C53, C54, C55, C56: DIGIKEY (none) -> 1189-2158-ND; LCSC (none) -> C413657; TYPE (none) -> EXT
- C61, C63, C64, C65, C66, C67, C68, C69, C70, C72, C89: LCSC (none) -> C15849; TYPE (none) -> BASIC
- C73, C74, C75, C91: footprint Capacitor_SMD:C_0603_1608Metric -> Capacitor_SMD:C_0805_2012Metric; LCSC (none) -> C15850; TYPE (none) -> BASIC
- C90: LCSC (none) -> C14663; TYPE (none) -> BASIC
- D1, D2, D3, D4: LCSC (none) -> C35722; TYPE (none) -> BASIC
- F1, F2, F3, F5: DIGIKEY (none) -> PTR030V0500-BK-ND; TYPE (none) -> DIGIKEY
- J4: DIGIKEY (none) -> WM4900-ND; TYPE (none) -> DIGIKEY
- L1: value 68uH/3A -> 68uH/2A; LCSC (none) -> C497902; TYPE (none) -> EXT
- L2, L3, L4: LCSC (none) -> C497902; TYPE (none) -> EXT
- R6, R9: LCSC (none) -> C25804; TYPE (none) -> BASIC
- U10, U6, U7, U8, U9: LCSC (none) -> C6186; TYPE (none) -> BASIC
- U11, U12, U21: LCSC (none) -> C20897; TYPE (none) -> BASIC
- U19: LCSC (none) -> C6185; TYPE (none) -> EXT
- U2, U3, U4, U5: LCSC (none) -> C61063; TYPE (none) -> BASIC
- U20: LCSC (none) -> C131103; TYPE (none) -> EXT

Commit message: Finished re-routing the power and important connections. exported dsn for this stage of routing. running autorouter, may have few more commits before finished route
Parts:
- F1, F2, F3, F5: footprint Fuse:Fuse_1206_3216Metric -> Capacitor_THT:C_Rect_L4.0mm_W2.5mm_P2.50mm
Changed lines of the file:
@@
 F 0 "F1" V 8645 2750 50  0000 C CNN
 F 1 "5A" V 8736 2750 50  0000 C CNN
-F 2 "Fuse:Fuse_1206_3216Metric" H 8900 2550 50  0001 L CNN
+F 2 "Capacitor_THT:C_Rect_L4.0mm_W2.5mm_P2.50mm" H 8900 2550 50  0001 L CNN
 F 3 "~" H 8850 2750 50  0001 C CNN
 F 4 "PTR030V0500-BK-ND" H 8850 2750 50  0001 C CNN "DIGIKEY"
@@
 F 0 "F2" V 8695 3850 50  0000 C CNN
 F 1 "5A" V 8786 3850 50  0000 C CNN
-F 2 "Fuse:Fuse_1206_3216Metric" H 8950 3650 50  0001 L CNN
+F 2 "Capacitor_THT:C_Rect_L4.0mm_W2.5mm_P2.50mm" H 8950 3650 50  0001 L CNN
 F 3 "~" H 8900 3850 50  0001 C CNN
 F 4 "PTR030V0500-BK-ND" H 8900 3850 50  0001 C CNN "DIGIKEY"
@@
 F 0 "F5" V 10545 3850 50  0000 C CNN
 F 1 "5A" V 10636 3850 50  0000 C CNN
-F 2 "Fuse:Fuse_1206_3216Metric" H 10800 3650 50  0001 L CNN
+F 2 "Capacitor_THT:C_Rect_L4.0mm_W2.5mm_P2.50mm" H 10800 3650 50  0001 L CNN
 F 3 "~" H 10750 3850 50  0001 C CNN
 F 4 "PTR030V0500-BK-ND" H 10750 3850 50  0001 C CNN "DIGIKEY"
@@
 F 0 "F3" V 10545 2800 50  0000 C CNN
 F 1 "5A" V 10636 2800 50  0000 C CNN
-F 2 "Fuse:Fuse_1206_3216Metric" H 10800 2600 50  0001 L CNN
+F 2 "Capacitor_THT:C_Rect_L4.0mm_W2.5mm_P2.50mm" H 10800 2600 50  0001 L CNN
 F 3 "~" H 10750 2800 50  0001 C CNN
 F 4 "PTR030V0500-BK-ND" H 10750 2800 50  0001 C CNN "DIGIKEY"

Commit message: updated bom with lcsc part #
Parts:
- C49, C50, C51, C52: DIGIKEY 399-18277-1-ND -> (none)
- C53, C54, C55, C56: DIGIKEY 1189-2158-ND -> (none)
- J4: LCSC (none) -> C239384; TYPE DIGIKEY -> EXT
Changed lines of the file:
@@
 F 3 "~" H 1200 1700 50  0001 C CNN
 F 4 "C3350" H 1200 1700 50  0001 C CNN "LCSC"
-F 5 "399-18277-1-ND" H 1200 1700 50  0001 C CNN "DIGIKEY"
+F 5 "" H 1200 1700 50  0001 C CNN "DIGIKEY"
 F 6 "EXT" H 1200 1700 50  0001 C CNN "TYPE"
 	1    1200 1700
@@
 F 3 "~" H 2750 1700 50  0001 C CNN
 F 4 "C413657" H 2750 1700 50  0001 C CNN "LCSC"
-F 5 "1189-2158-ND" H 2750 1700 50  0001 C CNN "DIGIKEY"
+F 5 "" H 2750 1700 50  0001 C CNN "DIGIKEY"
 F 6 "EXT" H 2750 1700 50  0001 C CNN "TYPE"
 	1    2750 1700
@@
 F 3 "~" H 1200 3600 50  0001 C CNN
 F 4 "C3350" H 1200 3600 50  0001 C CNN "LCSC"
-F 5 "399-18277-1-ND" H 1200 3600 50  0001 C CNN "DIGIKEY"
+F 5 "" H 1200 3600 50  0001 C CNN "DIGIKEY"
 F 6 "EXT" H 1200 3600 50  0001 C CNN "TYPE"
 	1    1200 3600
@@
 F 3 "~" H 2750 3600 50  0001 C CNN
 F 4 "C413657" H 2750 3600 50  0001 C CNN "LCSC"
-F 5 "1189-2158-ND" H 2750 3600 50  0001 C CNN "DIGIKEY"
+F 5 "" H 2750 3600 50  0001 C CNN "DIGIKEY"
 F 6 "EXT" H 2750 3600 50  0001 C CNN "TYPE"
 	1    2750 3600
@@
 F 3 "~" H 1150 5400 50  0001 C CNN
 F 4 "C3350" H 1150 5400 50  0001 C CNN "LCSC"
-F 5 "399-18277-1-ND" H 1150 5400 50  0001 C CNN "DIGIKEY"
+F 5 "" H 1150 5400 50  0001 C CNN "DIGIKEY"
 F 6 "EXT" H 1150 5400 50  0001 C CNN "TYPE"
 	1    1150 5400
@@
 F 3 "~" H 2700 5400 50  0001 C CNN
 F 4 "C413657" H 2700 5400 50  0001 C CNN "LCSC"
-F 5 "1189-2158-ND" H 2700 5400 50  0001 C CNN "DIGIKEY"
+F 5 "" H 2700 5400 50  0001 C CNN "DIGIKEY"
 F 6 "EXT" H 2700 5400 50  0001 C CNN "TYPE"
 	1    2700 5400
@@
 F 3 "~" H 1050 7150 50  0001 C CNN
 F 4 "C3350" H 1050 7150 50  0001 C CNN "LCSC"
-F 5 "399-18277-1-ND" H 1050 7150 50  0001 C CNN "DIGIKEY"
+F 5 "" H 1050 7150 50  0001 C CNN "DIGIKEY"
 F 6 "EXT" H 1050 7150 50  0001 C CNN "TYPE"
 	1    1050 7150
@@
 F 3 "~" H 2600 7150 50  0001 C CNN
 F 4 "C413657" H 2600 7150 50  0001 C CNN "LCSC"
-F 5 "1189-2158-ND" H 2600 7150 50  0001 C CNN "DIGIKEY"
+F 5 "" H 2600 7150 50  0001 C CNN "DIGIKEY"
 F 6 "EXT" H 2600 7150 50  0001 C CNN "TYPE"
 	1    2600 7150
@@
 F 3 "~" H 9700 1050 50  0001 C CNN
 F 4 "WM4900-ND" H 9700 1050 50  0001 C CNN "DIGIKEY"
-F 5 "DIGIKEY" H 9700 1050 50  0001 C CNN "TYPE"
+F 5 "EXT" H 9700 1050 50  0001 C CNN "TYPE"
+F 6 "C239384" H 9700 1050 50  0001 C CNN "LCSC"
 	1    9700 1050
 	1    0    0    -1

Commit message: added more functionality to JSON for motion quartet, motion set, motion profiles, machine profile, and more
Parts:
- C140, C141, C142, C49, C50, C51, C52, C53, C54, C55, C56, C57, C58, C59, C60, C61, C62, C63, C64, C65, C66, C67, C68, C69, C70, C71, C72, C73, C74, C75, C88, C89, C90, C91, D1, D2, D3, D4, L1, L2, L3, L4, R6, R9, U10, U11, U12, U2, U21, U3, U4, U5, U6, U7, U8, U9: ASSEMBLED (none) -> YES
- F1, F2, F3, F5, J4, U19, U20: ASSEMBLED (none) -> NO
