File: Hardware/MAD_P2/Power2.sch (KiCad schematic (older format))
At the start: 93 parts, among them J1 Line_1_3, J12 Line_3_3, J17 Line_1_2, J2 Line_2_2, J27 Line_1_1, J28 Line_2_1, J29 Line_2_3, J3 Line_3_1, J30 Line_3_2, U13 XL1509-5.0, U14 XL1509-5.0, U15 AMS1117-3.3, U16 AMS1117-3.3, U18 AMS1117-3.3, U22 XL1509-5.0, U24 AMS1117-3.3

Commit message: updated bom with lcsc part #
Parts:
- C76, C77, C92: DIGIKEY 399-18277-1-ND -> (none)
- C78, C79, C93: DIGIKEY 1189-2158-ND -> (none)
- J1, J12, J17, J2, J27, J28, J29, J3, J30: LCSC (none) -> C239384; TYPE DIGIKEY -> EXT
Changed lines of the file:
@@
 F 3 "~" H 1200 2050 50  0001 C CNN
 F 4 "C3350" H 1200 2050 50  0001 C CNN "LCSC"
-F 5 "399-18277-1-ND" H 1200 2050 50  0001 C CNN "DIGIKEY"
+F 5 "" H 1200 2050 50  0001 C CNN "DIGIKEY"
 F 6 "EXT" H 1200 2050 50  0001 C CNN "TYPE"
 	1    1200 2050
@@
 F 3 "~" H 2750 2050 50  0001 C CNN
 F 4 "C413657" H 2750 2050 50  0001 C CNN "LCSC"
-F 5 "1189-2158-ND" H 2750 2050 50  0001 C CNN "DIGIKEY"
+F 5 "" H 2750 2050 50  0001 C CNN "DIGIKEY"
 F 6 "EXT" H 2750 2050 50  0001 C CNN "TYPE"
 	1    2750 2050
@@
 F 3 "~" H 1100 6100 50  0001 C CNN
 F 4 "C3350" H 1100 6100 50  0001 C CNN "LCSC"
-F 5 "399-18277-1-ND" H 1100 6100 50  0001 C CNN "DIGIKEY"
+F 5 "" H 1100 6100 50  0001 C CNN "DIGIKEY"
 F 6 "EXT" H 1100 6100 50  0001 C CNN "TYPE"
 	1    1100 6100
@@
 F 3 "~" H 2650 6100 50  0001 C CNN
 F 4 "C413657" H 2650 6100 50  0001 C CNN "LCSC"
-F 5 "1189-2158-ND" H 2650 6100 50  0001 C CNN "DIGIKEY"
+F 5 "" H 2650 6100 50  0001 C CNN "DIGIKEY"
 F 6 "EXT" H 2650 6100 50  0001 C CNN "TYPE"
 	1    2650 6100
@@
 F 3 "~" H 2750 4200 50  0001 C CNN
 F 4 "C413657" H 2750 4200 50  0001 C CNN "LCSC"
-F 5 "1189-2158-ND" H 2750 4200 50  0001 C CNN "DIGIKEY"
+F 5 "" H 2750 4200 50  0001 C CNN "DIGIKEY"
 F 6 "EXT" H 2750 4200 50  0001 C CNN "TYPE"
 	1    2750 4200
@@
 F 3 "~" H 1200 4200 50  0001 C CNN
 F 4 "C3350" H 1200 4200 50  0001 C CNN "LCSC"
-F 5 "399-18277-1-ND" H 1200 4200 50  0001 C CNN "DIGIKEY"
+F 5 "" H 1200 4200 50  0001 C CNN "DIGIKEY"
 F 6 "EXT" H 1200 4200 50  0001 C CNN "TYPE"
 	1    1200 4200
@@
 F 3 "~" H 10650 1200 50  0001 C CNN
 F 4 "WM4900-ND" H 10650 1200 50  0001 C CNN "DIGIKEY"
-F 5 "DIGIKEY" H 10650 1200 50  0001 C CNN "TYPE"
+F 5 "EXT" H 10650 1200 50  0001 C CNN "TYPE"
+F 6 "C239384" H 10650 1200 50  0001 C CNN "LCSC"
 	1    10650 1200
 	1    0    0    -1
@@
 F 3 "~" H 10650 3500 50  0001 C CNN
 F 4 "WM4900-ND" H 10650 3500 50  0001 C CNN "DIGIKEY"
-F 5 "DIGIKEY" H 10650 3500 50  0001 C CNN "TYPE"
+F 5 "EXT" H 10650 3500 50  0001 C CNN "TYPE"
+F 6 "C239384" H 10650 3500 50  0001 C CNN "LCSC"
 	1    10650 3500
 	1    0    0    -1
@@
 F 3 "~" H 8650 4500 50  0001 C CNN
 F 4 "WM4900-ND" H 8650 4500 50  0001 C CNN "DIGIKEY"
-F 5 "DIGIKEY" H 8650 4500 50  0001 C CNN "TYPE"
+F 5 "EXT" H 8650 4500 50  0001 C CNN "TYPE"
+F 6 "C239384" H 8650 4500 50  0001 C CNN "LCSC"
 	1    8650 4500
 	1    0    0    -1
@@
 F 3 "~" H 10600 2300 50  0001 C CNN
 F 4 "WM4900-ND" H 10600 2300 50  0001 C CNN "DIGIKEY"
-F 5 "DIGIKEY" H 10600 2300 50  0001 C CNN "TYPE"
+F 5 "EXT" H 10600 2300 50  0001 C CNN "TYPE"
+F 6 "C239384" H 10600 2300 50  0001 C CNN "LCSC"
 	1    10600 2300
 	1    0    0    -1
@@
 F 3 "~" H 8600 2050 50  0001 C CNN
 F 4 "WM4900-ND" H 8600 2050 50  0001 C CNN "DIGIKEY"
-F 5 "DIGIKEY" H 8600 2050 50  0001 C CNN "TYPE"
+F 5 "EXT" H 8600 2050 50  0001 C CNN "TYPE"
+F 6 "C239384" H 8600 2050 50  0001 C CNN "LCSC"
 	1    8600 2050
 	1    0    0    -1
@@
 F 3 "~" H 8600 3300 50  0001 C CNN
 F 4 "WM4900-ND" H 8600 3300 50  0001 C CNN "DIGIKEY"
-F 5 "DIGIKEY" H 8600 3300 50  0001 C CNN "TYPE"
+F 5 "EXT" H 8600 3300 50  0001 C CNN "TYPE"
+F 6 "C239384" H 8600 3300 50  0001 C CNN "LCSC"
 	1    8600 3300
 	1    0    0    -1
@@
 F 3 "~" H 10650 4700 50  0001 C CNN
 F 4 "WM4900-ND" H 10650 4700 50  0001 C CNN "DIGIKEY"
-F 5 "DIGIKEY" H 10650 4700 50  0001 C CNN "TYPE"
+F 5 "EXT" H 10650 4700 50  0001 C CNN "TYPE"
+F 6 "C239384" H 10650 4700 50  0001 C CNN "LCSC"
 	1    10650 4700
 	1    0    0    -1
@@
 F 3 "~" H 10700 5900 50  0001 C CNN
 F 4 "WM4900-ND" H 10700 5900 50  0001 C CNN "DIGIKEY"
-F 5 "DIGIKEY" H 10700 5900 50  0001 C CNN "TYPE"
+F 5 "EXT" H 10700 5900 50  0001 C CNN "TYPE"
+F 6 "C239384" H 10700 5900 50  0001 C CNN "LCSC"
 	1    10700 5900
 	1    0    0    -1
@@
 F 3 "~" H 8650 5600 50  0001 C CNN
 F 4 "WM4900-ND" H 8650 5600 50  0001 C CNN "DIGIKEY"
-F 5 "DIGIKEY" H 8650 5600 50  0001 C CNN "TYPE"
+F 5 "EXT" H 8650 5600 50  0001 C CNN "TYPE"
+F 6 "C239384" H 8650 5600 50  0001 C CNN "LCSC"
 	1    8650 5600
 	1    0    0    -1

Commit message: added more functionality to JSON for motion quartet, motion set, motion profiles, machine profile, and more
Parts:
- C100, C101, C76, C77, C78, C79, C80, C81, C82, C83, C84, C85, C86, C87, C92, C93, C95, C97, D10, D11, D13, D14, D15, D16, D17, D18, D19, D20, D21, D22, D5, D6, D7, D8, L10, L11, L6, R12, R13, R25, R3, R30, R31, R32, R33, R34, R4, R5, R7, R8, U13, U14, U15, U16, U18, U22, U24: ASSEMBLED (none) -> YES
- J1, J12, J17, J2, J27, J28, J29, J3, J30: ASSEMBLED (none) -> NO
