File: Hardware/MAD_P2/MAD_P2.kicad_pcb (KiCad board)
At the start: 4 copper layers, 121.6 x 145.5 mm, 364 parts, among them J1 Line_1_3, J10 Conn_02x05_Odd_Even, J11 Conn_02x05_Odd_Even, J12 Line_3_3, J13 Conn_02x05_Odd_Even, J14 Conn_02x05_Odd_Even, J15 Conn_ADC1, J16 Conn_DAC, J17 Line_1_2, J18 P3, J19 P4, J2 Line_2_2, J20 P2, J21 Conn_02x05_Odd_Even, J22 Conn_02x05_Odd_Even, J23 Conn_02x03_Odd_Even, J24 P5, J25 P6, J26 P7, J27 Line_1_1, J28 Line_2_1, J29 Line_2_3, J3 Line_3_1, J30 Line_3_2, J31 Micro_SD_Card_Connector, J32 Micro_SD_Card_Socket, J33 Shifted IO, J34 FTDI 1x6, J4 Power_In, J5 Micro_SD_Card, J6 Edge_Conn, J7 Conn_02x05_Odd_Even, J8 USB_C_Receptacle_USB2.0, J9 Conn_02x05_Odd_Even, P10 CONN_01X01, P11 CONN_01X01, P13 CONN_01X01, P8 CONN_01X01, Q1 MMBT3904, Q2 2N7002, Q3 2N7002, Q4 2N7002, Q5 2N7002, SW1 Switch_SW_Push, U1 P2X8C4M64P-REF, U10 AMS1117-3.3, U11 APM4953, U12 APM4953, U13 XL1509-5.0, U14 XL1509-5.0, U15 AMS1117-3.3, U16 AMS1117-3.3, U17 MAX5134-7, U18 AMS1117-3.3, U19 AMS1117-1.8, U2 XL1509-5.0, U20 LM321, U21 APM4953, U22 XL1509-5.0, U23 ADS131A04, U24 AMS1117-3.3, U26 W25Q128JVS, U27 FT232RL, U28 DS3231M, U29 ESP-12F, U3 XL1509-5.0, U4 XL1509-5.0, U5 XL1509-5.0, U6 AMS1117-3.3, U7 AMS1117-3.3, U8 AMS1117-3.3, U9 AMS1117-3.3, Y1 20MHz, Y2 16.384MHz

Commit message: board complete, exporting production files
Parts:
- added DISP_HOLE_1: Hole_5.08, Tensile_Board:Hole_5.08, F.Cu at (395.6, 18.4)
- added DISP_HOLE_3: Hole_5.08, Tensile_Board:Hole_5.08, F.Cu at (395.6, 157.9)
Routing:
- net P7: track 0.00 -> 249.8 mm, vias 0 -> 4
- net RESET: track 16.9 -> 260.5 mm, vias 0 -> 5
- net P36: track 0.00 -> 230.1 mm, vias 0 -> 3
- net P62: track 0.00 -> 217.1 mm, vias 0 -> 3
- net P55: track 0.00 -> 206.8 mm, vias 0 -> 3
- net P63: track 0.00 -> 199.8 mm, vias 0 -> 3
- net P44: track 0.00 -> 199.1 mm, vias 0 -> 3
- net P47: track 0.00 -> 198.8 mm, vias 0 -> 4
- net P45: track 0.00 -> 196.1 mm, vias 0 -> 5
- net P42: track 0.00 -> 190.8 mm, vias 0 -> 4
- net P35: track 0.00 -> 185.4 mm, vias 0 -> 4
- net P41: track 0.00 -> 181.5 mm, vias 0 -> 4
- net P49: track 0.00 -> 176.3 mm, vias 0 -> 5
- net P40: track 0.00 -> 176.2 mm, vias 0 -> 4
- net P54: track 1.67 -> 176.7 mm, vias 0 -> 4
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- added copper zone on F.Cu, net (none)
- removed copper zone on In1.Cu, net 3.3V_ADC
Other:
- board text removed: "***WARNING***"
- board text removed: "BOTTOM_FRONT"
- board text removed: "INNER_FRONT"
- board text removed: "OUTER_FRONT"
- board text removed: "TOP_FRONT"

Commit message: syncing info
Other:
- net class Default removed
